File: swd2usbc-basic/swd2usbc-basic.kicad_sch (KiCad schematic)
At the start: 5 parts, among them J1 USB_C_Receptacle, J2 Conn_ARM_JTAG_SWD_10, J3 USB_C_Receptacle

Commit message: Adding swd2usbc and renaming swd2usbc-basic
Parts:
- J2: LCSC C2935458 -> C19191729
Other:
- company: Quesadillon LLC -> alvarop.com
- title: Debugotron - SWD2USBC -> SWD2USBC Basic
Changed lines of the file:
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@@
 	(paper "A4")
 	(title_block
-		(title "Debugotron - SWD2USBC")
-		(date "2024-12-31")
+		(title "SWD2USBC Basic")
+		(date "2025-01-05")
 		(rev "4.1")
-		(company "Quesadillon LLC")
+		(company "alvarop.com")
 	)
 	(junction
@@
 			)
 		)
-		(property "LCSC" "C2935458"
+		(property "LCSC" "C19191729"
 			(at 138.43 100.3299 0)
 			(effects

Commit message: Various fixes while ordering from JLCPCB
Parts:
- D1: LCSC C72043 -> C965804
Changed lines of the file:
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@@
 			)
 		)
-		(property "LCSC" "C72043"
+		(property "LCSC" "C965804"
 			(at 152.3365 52.07 0)
 			(effects
