File: swd2usbc/swd2usbc.kicad_sch (KiCad schematic)
At the start: 16 parts, among them J1 USB_C_Receptacle_USB2.0, J2 Conn_ARM_JTAG_SWD_10, P1 USB_C_Plug, U1 ATtiny24-20M

Commit message: Various fixes while ordering from JLCPCB
Parts:
- D1: LCSC C72043 -> C965804
- J2: LCSC C19191729 -> C2935458
- U1: LCSC C220282 -> C617902
Changed lines of the file:
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@@
 			)
 		)
-		(property "LCSC" "C72043"
+		(property "LCSC" "C965804"
 			(at 182.8165 87.63 0)
 			(effects
@@
 			)
 		)
-		(property "LCSC" "C19191729"
+		(property "LCSC" "C2935458"
 			(at 110.49 158.7499 0)
 			(effects
@@
 			)
 		)
-		(property "LCSC" "C220282"
+		(property "LCSC" "C617902"
 			(at 107.95 57.1499 0)
 			(effects
