File: sample-target/sample-target.kicad_pcb (KiCad board)
At the start: 4 copper layers, 51.8 x 20 mm, 56 parts, among them J1 USB_C_Receptacle, J2 Conn_01x03, SW1 SW_Push, SW2 SW_Push, U1 MIC5504-3.3YM5, U2 W25Q128JVS, U3 RP2040, U4 LM358_DFN, U5 SN74AHC1G08DBVR, U6 TMUX1511PWR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

Commit message: Add CC lines to sample targets
Connections:
- U3 pad 38: unconnected-(U3-GPIO26_ADC0-Pad38) -> /CC2
- U3 pad 40: unconnected-(U3-GPIO28_ADC2-Pad40) -> /CC1
Routing:
- net /CC2: track 11.8 -> 74.6 mm, vias 1 -> 3
- net /CC1: track 9.14 -> 52.9 mm, vias 2 -> 3

Commit message: Add pull up resistor to spi flash
Parts:
- added R12: 1k, Resistor_SMD:R_0402_1005Metric, F.Cu at (100.5, 105.4)
Routing:
- net /QSPI_SS: track 29.8 -> 31.1 mm
- net +3V3: track 34.3 -> 35.1 mm, vias 10 -> 11
