File: sample-target/sample-target.kicad_sch (KiCad schematic)
At the start: 46 parts, among them J1 USB_C_Receptacle, J2 Conn_01x03, SW1 SW_Push, SW2 SW_Push, U1 MIC5504-3.3YM5, U2 W25Q128JVS, U3 RP2040, U4 LM358_DFN, U5 SN74AHC1G08DBVR, U6 TMUX1511PWR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

Commit message: Various fixes while ordering from JLCPCB
Parts:
- J1: LCSC C134092 -> C2761408
Changed lines of the file:
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@@
 			)
 		)
-		(property "LCSC" "C134092"
+		(property "LCSC" "C2761408"
 			(at 45.72 71.12 0)
 			(effects

Commit message: Add CC lines to sample targets
Connections:
- net CC1: now also U3.40 (GPIO28_ADC2)
- net CC2: now also U3.38 (GPIO26_ADC0)
- no-connect marks 35 -> 33
Changed lines of the file:
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@@
 	(title_block
 		(title "SWD2USBC Sample Target")
-		(date "2025-01-05")
-		(rev "v1.0")
+		(date "2025-02-16")
+		(rev "v1.1")
 		(company "alvarop.com")
 	)
@@
 	)
 	(no_connect
-		(at 325.12 144.78)
-	)
-	(no_connect
 		(at 60.96 71.12)
 	)
@@
 	)
 	(no_connect
-		(at 325.12 139.7)
-	)
-	(no_connect
 		(at 60.96 88.9)
 	)
@@
 	(wire
 		(pts
+			(xy 325.12 144.78) (xy 331.47 144.78)
+		)
+		(stroke
+			(width 0)
+			(type default)
+		)
+	)
+	(wire
+		(pts
 			(xy 369.57 92.71) (xy 369.57 95.25)
 		)
@@
 	(wire
 		(pts
+			(xy 325.12 139.7) (xy 331.47 139.7)
+		)
+		(stroke
+			(width 0)
+			(type default)
+		)
+	)
+	(wire
+		(pts
 			(xy 304.8 60.96) (xy 304.8 63.5)
 		)
@@
 	(label "QSPI_SD3"
 		(at 259.08 101.6 0)
-		(fields_autoplaced yes)
 		(effects
 			(font
@@
 	(label "CC2"
 		(at 99.06 53.34 180)
-		(fields_autoplaced yes)
 		(effects
 			(font
@@
 	(label "CC2_AMP"
 		(at 74.93 172.72 180)
-		(fields_autoplaced yes)
 		(effects
 			(font
@@
 	(label "DAM_EN"
 		(at 121.92 162.56 180)
-		(fields_autoplaced yes)
 		(effects
 			(font
@@
 	(label "SWD"
 		(at 259.08 139.7 0)
-		(fields_autoplaced yes)
 		(effects
 			(font
@@
 	(label "USB_D+"
 		(at 236.22 73.66 0)
-		(fields_autoplaced yes)
 		(effects
 			(font
@@
 	(label "QSPI_SS"
 		(at 259.08 88.9 0)
-		(fields_autoplaced yes)
 		(effects
 			(font
@@
 	(label "SWD"
 		(at 200.66 147.32 180)
-		(fields_autoplaced yes)
 		(effects
 			(font
@@
 	(label "CC1"
 		(at 99.06 50.8 180)
-		(fields_autoplaced yes)
 		(effects
 			(font
@@
 	(label "QSPI_SD0"
 		(at 259.08 93.98 0)
-		(fields_autoplaced yes)
 		(effects
 			(font
@@
 	(label "SWDCLK_IN"
 		(at 142.24 152.4 0)
-		(fields_autoplaced yes)
 		(effects
 			(font
@@
 	(label "USB_D+"
 		(at 73.66 66.04 180)
-		(fields_autoplaced yes)
 		(effects
 			(font
@@
 	(label "SWDIO_IN"
 		(at 142.24 147.32 0)
-		(fields_autoplaced yes)
 		(effects
 			(font
@@
 	(label "GND_IN"
 		(at 73.66 104.14 180)
-		(fields_autoplaced yes)
 		(effects
 			(font
@@
 	(label "USB_D-"
 		(at 73.66 60.96 180)
-		(fields_autoplaced yes)
 		(effects
 			(font
@@
 	(label "SWO_IN"
 		(at 142.24 200.66 0)
-		(fields_autoplaced yes)
 		(effects
 			(font
@@
 	(label "RUN"
 		(at 259.08 71.12 0)
-		(fields_autoplaced yes)
 		(effects
 			(font
@@
 	(label "CC1"
 		(at 38.1 152.4 0)
-		(fields_autoplaced yes)
 		(effects
 			(font
@@
 	(label "XIN"
 		(at 259.08 116.84 0)
-		(fields_autoplaced yes)
 		(effects
 			(font
@@
 	(label "~{USB_BOOT}"
 		(at 287.02 215.9 0)
-		(fields_autoplaced yes)
 		(effects
 			(font
@@
 	(label "QSPI_SD3"
 		(at 313.69 228.6 0)
-		(fields_autoplaced yes)
 		(effects
 			(font
@@
 	(label "SWCLK"
 		(at 200.66 152.4 180)
-		(fields_autoplaced yes)
 		(effects
 			(font
@@
 	(label "QSPI_SCLK"
 		(at 313.69 218.44 0)
-		(fields_autoplaced yes)
 		(effects
 			(font
@@
 	(label "LED2"
 		(at 349.25 92.71 0)
-		(fields_autoplaced yes)
 		(effects
 			(font
@@
 	(label "SWDCLK_IN"
 		(at 73.66 78.74 180)
-		(fields_autoplaced yes)
+		(effects
+			(font
+				(size 1.27 1.27)
+			)
+			(justify right bottom)
+		)
+	)
+	(label "CC1"
+		(at 331.47 144.78 180)
 		(effects
 			(font
@@
 	(label "CC2"
 		(at 38.1 170.18 0)
-		(fields_autoplaced yes)
 		(effects
 			(font
@@
 		)
 	)
+	(label "CC2"
+		(at 331.47 139.7 180)
+		(effects
+			(font
+				(size 1.27 1.27)
+			)
+			(justify right bottom)
+		)
+	)
 	(label "XOUT"
 		(at 259.08 127 0)
-		(fields_autoplaced yes)
 		(effects
 			(font
@@
 	(label "UART0_TX"
 		(at 344.17 71.12 180)
-		(fields_autoplaced yes)
 		(effects
 			(font
@@
 	(label "GND_IN"
 		(at 142.24 149.86 0)
-		(fields_autoplaced yes)
 		(effects
 			(font
@@
 	(label "SWDIO_IN"
 		(at 73.66 81.28 180)
-		(fields_autoplaced yes)
 		(effects
 			(font
@@
 	(label "QSPI_SD2"
 		(at 259.08 99.06 0)
-		(fields_autoplaced yes)
 		(effects
 			(font
@@
 	(label "SWO"
 		(at 205.74 200.66 180)
-		(fields_autoplaced yes)
 		(effects
 			(font
@@
 	(label "UART0_RX"
 		(at 344.17 73.66 180)
-		(fields_autoplaced yes)
 		(effects
 			(font
@@
 	(label "RUN"
 		(at 278.13 215.9 180)
-		(fields_autoplaced yes)
 		(effects
 			(font
@@
 	(label "VREF"
 		(at 30.48 167.64 180)
-		(fields_autoplaced yes)
 		(effects
 			(font
@@
 	(label "LED1"
 		(at 349.25 82.55 0)
-		(fields_autoplaced yes)
 		(effects
 			(font
@@
 	(label "NRST_IN"
 		(at 142.24 198.12 0)
-		(fields_autoplaced yes)
 		(effects
 			(font
@@
 	(label "D-"
 		(at 262.89 83.82 0)
-		(fields_autoplaced yes)
 		(effects
 			(font
@@
 	(label "NRST_IN"
 		(at 73.66 96.52 180)
-		(fields_autoplaced yes)
 		(effects
 			(font
@@
 	(label "VTARGET_IN"
 		(at 73.66 101.6 180)
-		(fields_autoplaced yes)
 		(effects
 			(font
@@
 	(label "XOUT"
 		(at 320.04 191.77 180)
-		(fields_autoplaced yes)
 		(effects
 			(font
@@
 	(label "D+"
 		(at 262.89 73.66 0)
-		(fields_autoplaced yes)
 		(effects
 			(font
@@
 	(label "SWCLK"
 		(at 259.08 137.16 0)
-		(fields_autoplaced yes)
 		(effects
 			(font
@@
 	(label "RUN"
 		(at 205.74 198.12 180)
-		(fields_autoplaced yes)
 		(effects
 			(font
@@
 	(label "SWO_IN"
 		(at 73.66 93.98 180)
-		(fields_autoplaced yes)
 		(effects
 			(font
@@
 	(label "QSPI_SD1"
 		(at 313.69 223.52 0)
-		(fields_autoplaced yes)
 		(effects
 			(font
@@
 	(label "CC1_AMP"
 		(at 74.93 154.94 180)
-		(fields_autoplaced yes)
 		(effects
 			(font
@@
 	(label "QSPI_SS"
 		(at 313.69 215.9 0)
-		(fields_autoplaced yes)
 		(effects
 			(font
@@
 	(label "USB_D-"
 		(at 236.22 83.82 0)
-		(fields_autoplaced yes)
 		(effects
 			(font
@@
 	(label "QSPI_SD1"
 		(at 259.08 96.52 0)
-		(fields_autoplaced yes)
 		(effects
 			(font
@@
 	(label "XIN"
 		(at 320.04 181.61 180)
-		(fields_autoplaced yes)
 		(effects
 			(font
@@
 	(label "VTARGET_IN"
 		(at 142.24 193.04 0)
-		(fields_autoplaced yes)
 		(effects
 			(font
@@
 	(label "QSPI_SD2"
 		(at 313.69 226.06 0)
-		(fields_autoplaced yes)
 		(effects
 			(font
@@
 	(label "QSPI_SD0"
 		(at 313.69 220.98 0)
-		(fields_autoplaced yes)
 		(effects
 			(font
@@
 	(label "QSPI_SCLK"
 		(at 259.08 104.14 0)
-		(fields_autoplaced yes)
 		(effects
 			(font

Commit message: Add pull up resistor to spi flash
Parts:
- added R12: 1k, Resistor_SMD:R_0402_1005Metric, symbol Device:R
Connections:
- net +3V3: now also R12.1
- net QSPI_SS: now also R12.2
Changed lines of the file:
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@@
 	(title_block
 		(title "SWD2USBC Sample Target")
-		(date "2025-02-16")
-		(rev "v1.1")
+		(date "2025-02-19")
+		(rev "v1.2")
 		(company "alvarop.com")
 	)
@@
 	)
 	(junction
+		(at 325.12 215.9)
+		(diameter 0)
+		(color 0 0 0 0)
+	)
+	(junction
 		(at 358.14 41.91)
 		(diameter 0)
@@
 	)
 	(junction
+		(at 339.09 196.85)
+		(diameter 0)
+		(color 0 0 0 0)
+	)
+	(junction
 		(at 193.04 160.02)
 		(diameter 0)
@@
 	(wire
 		(pts
+			(xy 325.12 196.85) (xy 339.09 196.85)
+		)
+		(stroke
+			(width 0)
+			(type default)
+		)
+	)
+	(wire
+		(pts
+			(xy 325.12 215.9) (xy 328.93 215.9)
+		)
+		(stroke
+			(width 0)
+			(type default)
+		)
+	)
+	(wire
+		(pts
 			(xy 312.42 30.48) (xy 323.85 30.48)
 		)
@@
 	(wire
 		(pts
+			(xy 325.12 210.82) (xy 325.12 215.9)
+		)
+		(stroke
+			(width 0)
+			(type default)
+		)
+	)
+	(wire
+		(pts
 			(xy 358.14 39.37) (xy 358.14 41.91)
 		)
@@
 	(wire
 		(pts
-			(xy 309.88 215.9) (xy 328.93 215.9)
+			(xy 309.88 215.9) (xy 325.12 215.9)
 		)
 		(stroke
@@
 	(wire
 		(pts
+			(xy 325.12 203.2) (xy 325.12 196.85)
+		)
+		(stroke
+			(width 0)
+			(type default)
+		)
+	)
+	(wire
+		(pts
 			(xy 259.08 71.12) (xy 274.32 71.12)
 		)
@@
 					(unit 1)
 				)
+			)
+		)
+	)
+	(symbol
+		(lib_id "Device:R")
+		(at 325.12 207.01 0)
+		(unit 1)
+		(exclude_from_sim no)
+		(in_bom yes)
+		(on_board yes)
+		(dnp no)
+		(property "Reference" "R12"
+			(at 319.8622 207.01 90)
+			(effects
+				(font
+					(size 1.27 1.27)
+				)
+			)
+		)
+		(property "Value" "1k"
+			(at 322.1736 207.01 90)
+			(effects
+				(font
+					(size 1.27 1.27)
+				)
+			)
+		)
+		(property "Footprint" "Resistor_SMD:R_0402_1005Metric"
+			(at 323.342 207.01 90)
+			(effects
+				(font
+					(size 1.27 1.27)
+				)
+				(hide yes)
+			)
+		)
+		(property "Datasheet" "~"
+			(at 325.12 207.01 0)
+			(effects
+				(font
+					(size 1.27 1.27)
+				)
+				(hide yes)
+			)
+		)
+		(property "Description" ""
+			(at 325.12 207.01 0)
+			(effects
+				(font
+					(size 1.27 1.27)
+				)
+				(hide yes)
+			)
+		)
+		(property "LCSC" "C4190"
+			(at 325.12 207.01 0)
+			(effects
+				(font
+					(size 1.27 1.27)
+				)
+				(hide yes)
+			)
+		)
+		(pin "1"
+		)
+		(pin "2"
+		)
+		(instances
+			(project "sample-target"
+				(path "/f3846d6f-2066-409b-95b3-d044da1ab9d1"
+					(reference "R12")
+					(unit 1)
+				)
